File: 9VAdapator.sch (KiCad schematic (older format))
At the start: 6 parts, among them P1 CONN_2, P2 CONN_2, U1 LM7809ACT

Commit message: Version1.0
Parts:
- removed P1: CONN_2, symbol CONN_2
- added K1: CONN_3, symbol CONN_3
Connections:
- net at C1.1, C2.1, U1.1 (IN): now also K1.3 (P3)
- net at C1.2, C2.2, C3.2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: now also K1.1 (P1)
- no-connect marks 0 -> 1
Changed lines of the file:
@@
 LIBS:contrib
 LIBS:valves
+LIBS:9VAdapator-cache
 EELAYER 24 0
 EELAYER END
@@
 $EndComp
 $Comp
-L CONN_2 P1
-U 1 1 54C56D70
-P 1650 2600
-F 0 "P1" V 1600 2600 40  0000 C CNN
-F 1 "CONN_2" V 1700 2600 40  0000 C CNN
-F 2 "" H 1650 2600 60  0000 C CNN
-F 3 "" H 1650 2600 60  0000 C CNN
-	1    1650 2600
-	-1   0    0    1
-$EndComp
-$Comp
 L CONN_2 P2
 U 1 1 54C56D84
@@
 	3900 2700 3900 2800
 Connection ~ 3900 2800
+$Comp
+L CONN_3 K1
+U 1 1 54C5A9D4
+P 1650 2600
+F 0 "K1" V 1600 2600 50  0000 C CNN
+F 1 "CONN_3" V 1700 2600 40  0000 C CNN
+F 2 "" H 1650 2600 60  0000 C CNN
+F 3 "" H 1650 2600 60  0000 C CNN
+	1    1650 2600
+	-1   0    0    1
+$EndComp
+NoConn ~ 2000 2600
 $EndSCHEMATC
